File: ECAD/FluxpadKicad/Fluxpad.kicad_pcb (KiCad board)
At the start: 2 copper layers, 39 x 60 mm, 26 parts, among them SW1 SW_SPST, SW2 SW_SPST, SW3 PEC12R-4017F-N0024, U1 SeeeduinoXIAO, U2 DRV5056A3QDBZx Lekker, U3 DRV5056A3QDBZx Lekker

Commit message: jlcpcb version
Parts:
- added H1: MountingHole, Tang:JLCPCB Tooling Hole, F.Cu at (102.5, 67.0)
- added H2: MountingHole, Tang:JLCPCB Tooling Hole, F.Cu at (137.5, 123.0)
- added H3: MountingHole, Tang:JLCPCB Tooling Hole, F.Cu at (102.5, 105.0)
- D1, D2, D3, D4: value LED -> WHITE LED; footprint LED_SMD:LED_0603_1608Metric -> Tang:LED_1206_3216Metric_ReverseMount_Hole1.8x2.4mm; moved to B.Cu
- R1, R2, R3, R4: value 20 -> 22
- SW1, SW2: footprint Switch_Keyboard_Hotswap_Kailh:SW_Hotswap_Kailh_MX_1.00u -> Tang:SW_Hotswap_Kailh_MX_1.00u
- moved 3V3 6.53 mm to (132.2, 80.0)
- moved GND1 6.38 mm to (132.2, 83.8)
Routing:
- net +3V3: track 78.9 -> 83.7 mm
- net GND: track 20.4 -> 16.5 mm, vias 8 -> 23
- net Net-(D3-A): track 3.30 -> 2.38 mm, vias 1 -> 0
- net Net-(D4-A): track 3.15 -> 2.38 mm, vias 1 -> 0
- net Net-(D2-A): track 3.15 -> 2.38 mm, vias 1 -> 0
- net Net-(D1-A): track 3.00 -> 2.22 mm, vias 1 -> 0
- added copper zone on F.Cu, net GND
Other:
- board text added: "FLUXPAD"
- board text added: "REV J1 T.Wu"
- board text removed: "FLUXPAD Rev3 T.W."
